File: hw/design/LineInput.sch (KiCad schematic (older format))
At the start: 6 parts

Commit message: updated libraries, new xfmr
updated libraries, selected transformer and added to library/documentation
Parts:
- removed C? (x3): 47p, symbol Device:C
- removed F?: 1A, 5x20mm, 250VAC, symbol Device:Fuse
- removed T?: 5:1, symbol Device:Transformer_1P_1S
- added T?: A41-80-24, symbol pps_klib:A41-80-24
- SW?: value SW_SPST -> 1410-F110-P1F1-W14Q-1A; MfrNum (none) -> 1410-F110-P1F1-W14Q-1A
Connections:
- net labels added: LINEp_prot
- net labels removed: EARTH, LINE_E, LINEp_fused
- wire segments 26 -> 16
Other:
- note added: "Circuit-Breaker Rocker Switch"
- note added: "Place windings in series for higher voltage\nPlace windings in parallel for lower voltage\n80VA rating (any configuration)"
- note removed: "5:1 Transformer\nBasic Isolation"
- note removed: "Common mode choke?\nPut in part and DNI?"
- note removed: "To Do:\n- part #s for everything except caps\n- packages for everything\n"
- note removed: "X & Y\nCapacitors"
- moved on the sheet: SW?
Changed lines of the file:
@@
 $EndDescr
 $Comp
-L Device:Fuse F?
-U 1 1 5E80D36A
-P 4150 3200
-F 0 "F?" V 3953 3200 50  0000 C CNN
-F 1 "1A, 5x20mm, 250VAC" V 4044 3200 50  0000 C CNN
-F 2 "" V 4080 3200 50  0001 C CNN
-F 3 "~" H 4150 3200 50  0001 C CNN
-	1    4150 3200
-	0    1    1    0
-$EndComp
-$Comp
-L Device:C C?
-U 1 1 5E80D59B
-P 4650 3450
-F 0 "C?" H 4750 3500 50  0000 L CNN
-F 1 "47p" H 4750 3400 50  0000 L CNN
-F 2 "" H 4688 3300 50  0001 C CNN
-F 3 "~" H 4650 3450 50  0001 C CNN
-F 4 "Vishay_VY2470K29U2JS63V7" H 4650 3450 50  0001 C CNN "MfrNum"
-F 5 "440VAC" H 4750 3300 50  0000 L CNN "VRating"
-	1    4650 3450
+L Switch:SW_SPST SW?
+U 1 1 5E80E027
+P 4000 3200
+F 0 "SW?" H 4000 3435 50  0000 C CNN
+F 1 "1410-F110-P1F1-W14Q-1A" H 4000 3344 50  0000 C CNN
+F 2 "" H 4000 3200 50  0001 C CNN
+F 3 "" H 4000 3200 50  0001 C CNN
+F 4 "1410-F110-P1F1-W14Q-1A" H 4000 3200 50  0001 C CNN "MfrNum"
+	1    4000 3200
 	1    0    0    -1
 $EndComp
 Wire Wire Line
-	4300 3200 4650 3200
-Wire Wire Line
-	5100 3200 5100 3300
-Wire Wire Line
-	4650 3300 4650 3200
-Connection ~ 4650 3200
-Wire Wire Line
-	4650 3200 5100 3200
-Wire Wire Line
-	4350 3400 4350 3700
-Wire Wire Line
-	4350 3700 4650 3700
-Wire Wire Line
-	4650 3600 4650 3700
-Connection ~ 4650 3700
-Wire Wire Line
-	4650 3700 5450 3700
-Wire Wire Line
-	3200 3600 3100 3600
-Wire Wire Line
-	5450 3800 5450 3700
-Connection ~ 5450 3700
-Wire Wire Line
-	5450 3700 5850 3700
-Wire Wire Line
-	5100 3200 5850 3200
-Connection ~ 5100 3200
-Wire Wire Line
-	5450 4300 5450 4100
-Wire Wire Line
-	5100 3600 5100 4300
-Connection ~ 5100 4300
-Wire Wire Line
-	5100 4300 5450 4300
-Text Notes 5050 3000 0    50   ~ 0
-X & Y\nCapacitors
-Wire Wire Line
-	3200 3600 3200 4300
+	3100 3200 3800 3200
+Text HLabel 8650 3200 2    50   BiDi ~ 0
+P
+Text HLabel 8650 3600 2    50   BiDi ~ 0
+N
+Text HLabel 3100 3200 0    50   Input ~ 0
+LINE_P
+Text HLabel 3100 3600 0    50   Input ~ 0
+LINE_N
+Text Label 8300 3200 0    50   ~ 0
+P
+Text Label 8300 3600 0    50   ~ 0
+N
+Text Label 4750 3200 0    50   ~ 0
+LINEp_prot
+Text Label 3850 3600 0    50   ~ 0
+LINEn
 $Comp
-L Switch:SW_SPST SW?
-U 1 1 5E80E027
-P 3450 3200
-F 0 "SW?" H 3450 3435 50  0000 C CNN
-F 1 "SW_SPST" H 3450 3344 50  0000 C CNN
-F 2 "" H 3450 3200 50  0001 C CNN
-F 3 "" H 3450 3200 50  0001 C CNN
-	1    3450 3200
+L pps_klib:A41-80-24 T?
+U 1 1 5EC59277
+P 6800 3700
+F 0 "T?" H 6450 4350 50  0000 C CNN
+F 1 "A41-80-24" H 6650 3050 50  0000 C CNN
+F 2 "" H 6900 3800 50  0001 C CNN
+F 3 "" H 6900 3800 50  0001 C CNN
+	1    6800 3700
 	1    0    0    -1
 $EndComp
 Wire Wire Line
-	3100 3200 3250 3200
+	6250 3600 6000 3600
 Wire Wire Line
-	3650 3200 4000 3200
+	6150 3200 6150 3800
 Wire Wire Line
-	3100 3400 4350 3400
-$Comp
-L Device:Transformer_1P_1S T?
-U 1 1 5E80EDDA
-P 6350 3450
-F 0 "T?" H 6350 3828 50  0000 C CNN
-F 1 "5:1" H 6350 3737 50  0000 C CNN
-F 2 "" H 6350 3450 50  0001 C CNN
-F 3 "~" H 6350 3450 50  0001 C CNN
-	1    6350 3450
-	1    0    0    -1
-$EndComp
+	6150 3800 6250 3800
+Connection ~ 6150 3200
 Wire Wire Line
-	5850 3200 5850 3250
+	6150 3200 6250 3200
 Wire Wire Line
-	5850 3250 5950 3250
+	6000 3600 6000 4200
 Wire Wire Line
-	5850 3700 5850 3650
+	6000 4200 6250 4200
+Connection ~ 6000 3600
 Wire Wire Line
-	5850 3650 5950 3650
-Text Notes 6100 3950 0    50   ~ 0
-5:1 Transformer\nBasic Isolation
+	7500 3800 7350 3800
 Wire Wire Line
-	6750 3250 7500 3250
+	7950 3600 7950 4200
 Wire Wire Line
-	6750 3650 7500 3650
-Text HLabel 7500 3250 2    50   BiDi ~ 0
-P
-Text HLabel 7500 3650 2    50   BiDi ~ 0
-N
+	7950 4200 7350 4200
 Wire Wire Line
-	3200 4300 5100 4300
-Text HLabel 3100 3200 0    50   Input ~ 0
-LINE_P
-Text HLabel 3100 3400 0    50   Input ~ 0
-LINE_N
-Text HLabel 3100 3600 0    50   Input ~ 0
-LINE_E
-Text Notes 4550 2100 0    50   ~ 0
-Common mode choke?\nPut in part and DNI?
-Text Label 7150 3250 0    50   ~ 0
-P
-Text Label 7150 3650 0    50   ~ 0
-N
-Text Label 3900 4300 0    50   ~ 0
-EARTH
-$Comp
-L Device:C C?
-U 1 1 5EC17EEF
-P 5100 3450
-F 0 "C?" H 5200 3500 50  0000 L CNN
-F 1 "47p" H 5200 3400 50  0000 L CNN
-F 2 "" H 5138 3300 50  0001 C CNN
-F 3 "~" H 5100 3450 50  0001 C CNN
-F 4 "Vishay_VY2470K29U2JS63V7" H 5100 3450 50  0001 C CNN "MfrNum"
-F 5 "440VAC" H 5200 3300 50  0000 L CNN "VRating"
-	1    5100 3450
-	1    0    0    -1
-$EndComp
-$Comp
-L Device:C C?
-U 1 1 5EC17F17
-P 5450 3950
-F 0 "C?" H 5550 4000 50  0000 L CNN
-F 1 "47p" H 5550 3900 50  0000 L CNN
-F 2 "" H 5488 3800 50  0001 C CNN
-F 3 "~" H 5450 3950 50  0001 C CNN
-F 4 "Vishay_VY2470K29U2JS63V7" H 5450 3950 50  0001 C CNN "MfrNum"
-F 5 "440VAC" H 5550 3800 50  0000 L CNN "VRating"
-	1    5450 3950
-	1    0    0    -1
-$EndComp
-Text Notes 750  1050 0    50   ~ 0
-To Do:\n- part #s for everything except caps\n- packages for everything\n
-Text Label 4750 3200 0    50   ~ 0
-LINEp_fused
-Text Label 3850 3400 0    50   ~ 0
-LINEn
+	7950 3600 8650 3600
+Wire Wire Line
+	3100 3600 6000 3600
+Wire Wire Line
+	4200 3200 6150 3200
+Text Notes 3500 2650 0    50   ~ 0
+Circuit-Breaker Rocker Switch
+Text Notes 5700 4900 0    50   ~ 0
+Place windings in series for higher voltage\nPlace windings in parallel for lower voltage\n80VA rating (any configuration)
+Wire Wire Line
+	7350 3200 8650 3200
+Wire Wire Line
+	7500 3800 7500 3600
+Wire Wire Line
+	7500 3600 7350 3600
 $EndSCHEMATC
