File: hw/design/PrimarySW.sch (KiCad schematic (older format))
At the start: 26 parts

Commit message: updated libraries, new xfmr
updated libraries, selected transformer and added to library/documentation
Parts:
- removed U?: LT8653S, symbol RDSmith:LT8653S
- added U?: LT8653S, symbol pps_klib:LT8653S
Changed lines of the file:
@@
-	1    0    0    -1
-$EndComp
-$Comp
-L RDSmith:LT8653S U?
-U 1 1 5E88D513
-P 6150 4200
-F 0 "U?" H 6150 5277 100 0000 C CNN
-F 1 "LT8653S" H 6150 5111 100 0000 C CNN
-F 2 "" H 6150 4200 100 0001 C CNN
-F 3 "" H 6150 4200 100 0001 C CNN
-	1    6150 4200
 	1    0    0    -1
 $EndComp
@@
 	1    0    0    -1
 $EndComp
+$Comp
+L pps_klib:LT8653S U?
+U 1 1 5EC501A8
+P 6150 4200
+F 0 "U?" H 5800 5100 100 0000 C CNN
+F 1 "LT8653S" H 6150 4900 100 0000 C CNN
+F 2 "" H 6150 4200 100 0001 C CNN
+F 3 "" H 6150 4200 100 0001 C CNN
+	1    6150 4200
+	1    0    0    -1
+$EndComp

Commit message: more work
more PFC work, more LDO work, added secondary regulator sheet, expanded system power tree sim
Parts:
- added TP?: 5V, TestPoint:TestPoint_Keystone_5000-5004_Miniature, symbol Connector:TestPoint
- added TP?: SWout, TestPoint:TestPoint_Keystone_5000-5004_Miniature, symbol Connector:TestPoint
- added TP?: SWfb, TestPoint:TestPoint_Keystone_5000-5004_Miniature, symbol Connector:TestPoint
- added TP?: SWgood, TestPoint:TestPoint_Keystone_5000-5004_Miniature, symbol Connector:TestPoint
- added TP?: 5Vgood, TestPoint:TestPoint_Keystone_5000-5004_Miniature, symbol Connector:TestPoint
- added TP?: SWen, TestPoint:TestPoint_Keystone_5000-5004_Miniature, symbol Connector:TestPoint
Connections:
- net 5V: now also TP?.1
- net PriSW_EN: now also TP?.1
- net Vadj: now also TP?.1
- net Vout: now also TP?.1
- net PGOOD renamed SW_GOOD
- net SW_GOOD: now also TP?.1
- net PriSW_pg1 renamed 5V_GOOD
- net 5V_GOOD: now also TP?.1
Changed lines of the file:
@@
 $Descr A4 11693 8268
 encoding utf-8
-Sheet 4 7
+Sheet 4 8
 Title ""
 Date ""
@@
 5V
 Text HLabel 2900 2000 0    50   BiDi ~ 0
-PGOOD
+SW_GOOD
 $Comp
 L Device:C C?
@@
 	8250 4500 8250 4800
 Wire Wire Line
-	8250 4800 7350 4800
-Wire Wire Line
 	7350 4800 7350 4100
 Wire Wire Line
@@
 Connection ~ 7950 2950
 Wire Wire Line
-	7950 2950 8550 2950
+	7950 2950 8200 2950
 NoConn ~ 6150 5100
 $Comp
@@
 Connection ~ 8850 4000
 Wire Wire Line
-	8850 4000 8450 4000
+	8850 4000 8700 4000
 Wire Wire Line
 	8850 4400 8850 4500
@@
 Wire Wire Line
 	3250 2000 2900 2000
-Wire Wire Line
-	3250 2000 3650 2000
 Connection ~ 3250 2000
 Wire Wire Line
@@
 Wire Wire Line
 	5050 2200 5050 2300
-Wire Wire Line
-	3950 2000 4750 2000
 Text Notes 5500 1350 0    50   ~ 0
 "5V GOOD"\nIndicator
@@
 	1    0    0    -1
 $EndComp
+$Comp
+L Connector:TestPoint TP?
+U 1 1 5EC552E4
+P 8200 2700
+AR Path="/5E80D1C0/5EC552E4" Ref="TP?"  Part="1"
+AR Path="/5E80D210/5EC552E4" Ref="TP?"  Part="1"
+AR Path="/5E84FADE/5EC552E4" Ref="TP?"  Part="1"
+F 0 "TP?" H 8150 3000 50  0000 L CNN
+F 1 "5V" H 8150 2900 50  0000 L CNN
+F 2 "TestPoint:TestPoint_Keystone_5000-5004_Miniature" H 8400 2700 50  0001 C CNN
+F 3 "~" H 8400 2700 50  0001 C CNN
+	1    8200 2700
+	1    0    0    -1
+$EndComp
+Wire Wire Line
+	8200 2700 8200 2950
+Connection ~ 8200 2950
+Wire Wire Line
+	8200 2950 8550 2950
+$Comp
+L Connector:TestPoint TP?
+U 1 1 5EC6AB90
+P 8700 3850
+AR Path="/5E80D1C0/5EC6AB90" Ref="TP?"  Part="1"
+AR Path="/5E80D210/5EC6AB90" Ref="TP?"  Part="1"
+AR Path="/5E84FADE/5EC6AB90" Ref="TP?"  Part="1"
+F 0 "TP?" H 8650 4150 50  0000 L CNN
+F 1 "SWout" H 8650 4050 50  0000 L CNN
+F 2 "TestPoint:TestPoint_Keystone_5000-5004_Miniature" H 8900 3850 50  0001 C CNN
+F 3 "~" H 8900 3850 50  0001 C CNN
+	1    8700 3850
+	1    0    0    -1
+$EndComp
+Wire Wire Line
+	8700 3850 8700 4000
+Connection ~ 8700 4000
+Wire Wire Line
+	8700 4000 8450 4000
+$Comp
+L Connector:TestPoint TP?
+U 1 1 5EC6EACC
+P 8150 5000
+AR Path="/5E80D1C0/5EC6EACC" Ref="TP?"  Part="1"
+AR Path="/5E80D210/5EC6EACC" Ref="TP?"  Part="1"
+AR Path="/5E84FADE/5EC6EACC" Ref="TP?"  Part="1"
+F 0 "TP?" V 8150 5200 50  0000 L CNN
+F 1 "SWfb" V 8050 5050 50  0000 L CNN
+F 2 "TestPoint:TestPoint_Keystone_5000-5004_Miniature" H 8350 5000 50  0001 C CNN
+F 3 "~" H 8350 5000 50  0001 C CNN
+	1    8150 5000
+	0    -1   -1   0
+$EndComp
+Wire Wire Line
+	8150 5000 8250 5000
+Wire Wire Line
+	8250 5000 8250 4800
+Wire Wire Line
+	7350 4800 8250 4800
+Connection ~ 8250 4800
+$Comp
+L Connector:TestPoint TP?
+U 1 1 5EC8958A
+P 3150 2200
+AR Path="/5E80D1C0/5EC8958A" Ref="TP?"  Part="1"
+AR Path="/5E80D210/5EC8958A" Ref="TP?"  Part="1"
+AR Path="/5E84FADE/5EC8958A" Ref="TP?"  Part="1"
+F 0 "TP?" V 3104 2388 50  0000 L CNN
+F 1 "SWgood" V 3195 2388 50  0000 L CNN
+F 2 "TestPoint:TestPoint_Keystone_5000-5004_Miniature" H 3350 2200 50  0001 C CNN
+F 3 "~" H 3350 2200 50  0001 C CNN
+	1    3150 2200
+	0    -1   -1   0
+$EndComp
+$Comp
+L Connector:TestPoint TP?
+U 1 1 5EC8D251
+P 4300 2200
+AR Path="/5E80D1C0/5EC8D251" Ref="TP?"  Part="1"
+AR Path="/5E80D210/5EC8D251" Ref="TP?"  Part="1"
+AR Path="/5E84FADE/5EC8D251" Ref="TP?"  Part="1"
+F 0 "TP?" V 4254 2388 50  0000 L CNN
+F 1 "5Vgood" V 4345 2388 50  0000 L CNN
+F 2 "TestPoint:TestPoint_Keystone_5000-5004_Miniature" H 4500 2200 50  0001 C CNN
+F 3 "~" H 4500 2200 50  0001 C CNN
+	1    4300 2200
+	0    -1   -1   0
+$EndComp
+Wire Wire Line
+	3950 2000 4500 2000
+Wire Wire Line
+	4300 2200 4500 2200
+Wire Wire Line
+	4500 2200 4500 2000
+Connection ~ 4500 2000
+Wire Wire Line
+	4500 2000 4750 2000
+Wire Wire Line
+	3250 2200 3250 2000
+Wire Wire Line
+	3250 2000 3650 2000
+Wire Wire Line
+	3250 2200 3150 2200
+$Comp
+L Connector:TestPoint TP?
+U 1 1 5ECBD5AE
+P 4100 3950
+AR Path="/5E80D1C0/5ECBD5AE" Ref="TP?"  Part="1"
+AR Path="/5E80D210/5ECBD5AE" Ref="TP?"  Part="1"
+AR Path="/5E84FADE/5ECBD5AE" Ref="TP?"  Part="1"
+F 0 "TP?" V 4054 4138 50  0000 L CNN
+F 1 "SWen" V 4145 4138 50  0000 L CNN
+F 2 "TestPoint:TestPoint_Keystone_5000-5004_Miniature" H 4300 3950 50  0001 C CNN
+F 3 "~" H 4300 3950 50  0001 C CNN
+	1    4100 3950
+	0    1    1    0
+$EndComp
+Wire Wire Line
+	4100 3950 4000 3950
+Connection ~ 4000 3950
+Text HLabel 4150 2450 0    50   BiDi ~ 0
+5V_GOOD
+Wire Wire Line
+	4150 2450 4500 2450
+Wire Wire Line
+	4500 2450 4500 2200
+Connection ~ 4500 2200
 $EndSCHEMATC

Commit message: lots of work
expanded README doc, specifications, added secondary regulator circuit + symbol, more component specs added
Parts:
- added TP?: GND, TestPoint:TestPoint_Keystone_5000-5004_Miniature, symbol Connector:TestPoint
- C? (x2): footprint (none) -> Capacitor_SMD:C_1210_3225Metric_Pad1.42x2.65mm_HandSolder
- C?: footprint (none) -> Resistor_SMD:R_1206_3216Metric_Pad1.42x1.75mm_HandSolder
- R? (x2): footprint (none) -> Resistor_SMD:R_0603_1608Metric
- R?: value R_US -> 2940
- R?: value R_US -> 100k; footprint Resistor_SMD:R_0603_1608Metric -> Resistor_SMD:R_0805_2012Metric; Size (none) -> 0603
Connections:
- net GND: now also TP?.1
Other:
- note added: "EN set to 27V\nWCA: min/max = 25.9V / 28.1V\n(resistors 1%, ref 4%)"
- note added: "Power-Good\nPull-ups"
- moved on the sheet: TP?
Changed lines of the file:
@@
 F 0 "C?" H 7300 3300 50  0000 L CNN
 F 1 "22u" H 7300 3200 50  0000 L CNN
-F 2 "" H 7238 3050 50  0001 C CNN
+F 2 "Capacitor_SMD:C_1210_3225Metric_Pad1.42x2.65mm_HandSolder" H 7238 3050 50  0001 C CNN
 F 3 "~" H 7200 3200 50  0001 C CNN
 F 4 "TDK_C3225X5R1C226K250AA" H 7200 3200 50  0001 C CNN "MfrNum"
@@
 F 0 "C?" H 7650 4350 50  0000 L CNN
 F 1 "10u" H 7650 4250 50  0000 L CNN
-F 2 "" H 7588 4100 50  0001 C CNN
+F 2 "Resistor_SMD:R_1206_3216Metric_Pad1.42x1.75mm_HandSolder" H 7588 4100 50  0001 C CNN
 F 3 "~" H 7550 4250 50  0001 C CNN
 F 4 "Murata_GRT31CR61H106ME01" H 7550 4250 50  0001 C CNN "MfrNum"
@@
 F 0 "R?" H 8518 4296 50  0000 L CNN
 F 1 "205k" H 8518 4205 50  0000 L CNN
-F 2 "" V 8490 4240 50  0001 C CNN
+F 2 "Resistor_SMD:R_0603_1608Metric" V 8490 4240 50  0001 C CNN
 F 3 "~" H 8450 4250 50  0001 C CNN
 	1    8450 4250
@@
 F 0 "R?" H 8518 4796 50  0000 L CNN
 F 1 "11.5k" H 8518 4705 50  0000 L CNN
-F 2 "" V 8490 4740 50  0001 C CNN
+F 2 "Resistor_SMD:R_0603_1608Metric" V 8490 4740 50  0001 C CNN
 F 3 "~" H 8450 4750 50  0001 C CNN
 	1    8450 4750
@@
 P 3750 4150
 F 0 "R?" H 3500 4200 50  0000 L CNN
-F 1 "R_US" H 3500 4100 50  0000 L CNN
+F 1 "2940" H 3500 4100 50  0000 L CNN
 F 2 "Resistor_SMD:R_0603_1608Metric" V 3790 4140 50  0001 C CNN
 F 3 "~" H 3750 4150 50  0001 C CNN
@@
 P 3750 3750
 F 0 "R?" H 3500 3800 50  0000 L CNN
-F 1 "R_US" H 3500 3700 50  0000 L CNN
-F 2 "Resistor_SMD:R_0603_1608Metric" V 3790 3740 50  0001 C CNN
+F 1 "100k" H 3500 3700 50  0000 L CNN
+F 2 "Resistor_SMD:R_0805_2012Metric" V 3790 3740 50  0001 C CNN
 F 3 "~" H 3750 3750 50  0001 C CNN
+F 4 "0603" H 3500 3600 50  0000 L CNN "Size"
 	1    3750 3750
 	1    0    0    -1
@@
 F 0 "C?" H 7700 3300 50  0000 L CNN
 F 1 "22u" H 7700 3200 50  0000 L CNN
-F 2 "" H 7638 3050 50  0001 C CNN
+F 2 "Capacitor_SMD:C_1210_3225Metric_Pad1.42x2.65mm_HandSolder" H 7638 3050 50  0001 C CNN
 F 3 "~" H 7600 3200 50  0001 C CNN
 F 4 "TDK_C3225X5R1C226K250AA" H 7600 3200 50  0001 C CNN "MfrNum"
@@
 	-1   0    0    -1
 $EndComp
-$Comp
-L Device:C C?
-U 1 1 5EC2E4DE
-P 4900 5700
-F 0 "C?" H 5050 5800 50  0000 L CNN
-F 1 "5.1p" H 5050 5700 50  0000 L CNN
-F 2 "Capacitor_SMD:C_0603_1608Metric" H 4938 5550 50  0001 C CNN
-F 3 "~" H 4900 5700 50  0001 C CNN
-F 4 "10V" H 5050 5600 50  0000 L CNN "VRating"
-F 5 "0402" H 5050 5500 50  0000 L CNN "Size"
-	1    4900 5700
-	-1   0    0    -1
-$EndComp
 Text Label 7700 4800 0    50   ~ 0
 PriSW_fb
@@
 Text Label 5450 5150 0    50   ~ 0
 PriSW_vcc
-Text Label 4900 5250 0    50   ~ 0
+Text Label 5150 5200 1    50   ~ 0
 PriSW_comp
-Text Label 4650 4400 0    50   ~ 0
+Text Label 4950 4400 0    50   ~ 0
 PriSW_ss1
-Text Label 4650 4500 0    50   ~ 0
-PriSW_ss2
 Text Label 4000 3750 0    50   ~ 0
 PriSW_EN
@@
 Wire Wire Line
 	5550 4000 4900 4000
-Wire Wire Line
-	4900 3900 5550 3900
 Text Label 4900 3900 0    50   ~ 0
 PriSW_pg1
@@
 	3250 1450 3050 1450
 Wire Wire Line
-	3250 1450 3950 1450
-Wire Wire Line
 	3950 1450 3950 1600
-Connection ~ 3250 1450
-Text Label 3050 1450 0    50   ~ 0
-5V
 Wire Wire Line
 	3250 1900 3250 2000
@@
 Wire Wire Line
 	5050 2200 5050 2300
-Text Notes 5500 1350 0    50   ~ 0
+Text Notes 5450 1700 0    50   ~ 0
 "5V GOOD"\nIndicator
 $Comp
@@
 L Connector:TestPoint TP?
 U 1 1 5EC552E4
-P 8200 2700
+P 8200 2800
 AR Path="/5E80D1C0/5EC552E4" Ref="TP?"  Part="1"
 AR Path="/5E80D210/5EC552E4" Ref="TP?"  Part="1"
 AR Path="/5E84FADE/5EC552E4" Ref="TP?"  Part="1"
-F 0 "TP?" H 8150 3000 50  0000 L CNN
-F 1 "5V" H 8150 2900 50  0000 L CNN
-F 2 "TestPoint:TestPoint_Keystone_5000-5004_Miniature" H 8400 2700 50  0001 C CNN
-F 3 "~" H 8400 2700 50  0001 C CNN
-	1    8200 2700
-	1    0    0    -1
-$EndComp
-Wire Wire Line
-	8200 2700 8200 2950
+F 0 "TP?" H 8150 3100 50  0000 L CNN
+F 1 "5V" H 8150 3000 50  0000 L CNN
+F 2 "TestPoint:TestPoint_Keystone_5000-5004_Miniature" H 8400 2800 50  0001 C CNN
+F 3 "~" H 8400 2800 50  0001 C CNN
+	1    8200 2800
+	1    0    0    -1
+$EndComp
+Wire Wire Line
+	8200 2800 8200 2950
 Connection ~ 8200 2950
 Wire Wire Line
@@
 	4500 2450 4500 2200
 Connection ~ 4500 2200
+$Comp
+L Device:C C?
+U 1 1 5EC2E4DE
+P 4900 5700
+F 0 "C?" H 5050 5800 50  0000 L CNN
+F 1 "5.1p" H 5050 5700 50  0000 L CNN
+F 2 "Capacitor_SMD:C_0603_1608Metric" H 4938 5550 50  0001 C CNN
+F 3 "~" H 4900 5700 50  0001 C CNN
+F 4 "10V" H 5050 5600 50  0000 L CNN "VRating"
+F 5 "0402" H 5050 5500 50  0000 L CNN "Size"
+	1    4900 5700
+	-1   0    0    -1
+$EndComp
+Text Notes 2600 5050 0    50   ~ 0
+EN set to 27V\nWCA: min/max = 25.9V / 28.1V\n(resistors 1%, ref 4%)
+Wire Wire Line
+	4900 3900 5550 3900
+Connection ~ 3250 1450
+Wire Wire Line
+	3250 1450 3950 1450
+Text Label 3050 1450 0    50   ~ 0
+5V
+Text Label 4950 4500 0    50   ~ 0
+PriSW_ss2
+Text Notes 3450 950  0    50   ~ 0
+Power-Good\nPull-ups
+$Comp
+L Connector:TestPoint TP?
+U 1 1 5ECD266E
+P 1800 6300
+AR Path="/5E80D1C0/5ECD266E" Ref="TP?"  Part="1"
+AR Path="/5E80D210/5ECD266E" Ref="TP?"  Part="1"
+AR Path="/5E84FADE/5ECD266E" Ref="TP?"  Part="1"
+AR Path="/5ECFB146/5ECD266E" Ref="TP?"  Part="1"
+F 0 "TP?" H 1750 6600 50  0000 L CNN
+F 1 "GND" H 1750 6500 50  0000 L CNN
+F 2 "TestPoint:TestPoint_Keystone_5000-5004_Miniature" H 2000 6300 50  0001 C CNN
+F 3 "~" H 2000 6300 50  0001 C CNN
+	1    1800 6300
+	1    0    0    -1
+$EndComp
+Wire Wire Line
+	1800 6300 1800 6450
+Connection ~ 1800 6450
 $EndSCHEMATC

Commit message: more part numbers
Added manfacturer part numbers to ICs, added descriptions to symbols in library
Parts:
- U?: MfrNum (none) -> LT8653SEV
Changed lines of the file:
@@
 F 2 "" H 6150 4200 100 0001 C CNN
 F 3 "" H 6150 4200 100 0001 C CNN
+F 4 "LT8653SEV" H 6150 4200 50  0001 C CNN "MfrNum"
 	1    6150 4200
 	1    0    0    -1
