File: hw/design/SupplyAdj.sch (KiCad schematic (older format))
At the start: 17 parts

Commit message: updated libraries, new xfmr
updated libraries, selected transformer and added to library/documentation
Parts:
- removed U? (x3): LTC7106, symbol RDSmith:LTC7106
- added U? (x3): LTC7106, symbol pps_klib:LTC7106
Changed lines of the file:
@@
 SDA
-$Comp
-L RDSmith:LTC7106 U?
-U 1 1 5E95F425
-P 4850 1700
-F 0 "U?" H 4500 2150 50  0000 C CNN
-F 1 "LTC7106" H 5100 2150 50  0000 C CNN
-F 2 "" H 4850 1700 50  0001 C CNN
-F 3 "" H 4850 1700 50  0001 C CNN
-	1    4850 1700
-	1    0    0    -1
-$EndComp
-$Comp
-L RDSmith:LTC7106 U?
-U 1 1 5E95F45F
-P 4850 3850
-F 0 "U?" H 4500 4300 50  0000 C CNN
-F 1 "LTC7106" H 5100 4300 50  0000 C CNN
-F 2 "" H 4850 3850 50  0001 C CNN
-F 3 "" H 4850 3850 50  0001 C CNN
-	1    4850 3850
-	1    0    0    -1
-$EndComp
-$Comp
-L RDSmith:LTC7106 U?
-U 1 1 5E95F48D
-P 4900 6000
-F 0 "U?" H 4550 6450 50  0000 C CNN
-F 1 "LTC7106" H 5150 6450 50  0000 C CNN
-F 2 "" H 4900 6000 50  0001 C CNN
-F 3 "" H 4900 6000 50  0001 C CNN
-	1    4900 6000
-	1    0    0    -1
-$EndComp
 $Comp
 L power:GND #PWR?
@@
 Wire Wire Line
 	4350 900  4450 900
-Wire Wire Line
-	4750 900  4850 900
 Text Label 5200 900  2    50   ~ 0
 Vdd
@@
 Text Label 5250 5200 2    50   ~ 0
 Vdd
-Wire Wire Line
-	4850 1200 4850 900
-Connection ~ 4850 900
-Wire Wire Line
-	4850 900  5200 900
 Wire Wire Line
 	4850 3350 4850 3050
@@
 	1    0    0    -1
 $EndComp
+$Comp
+L pps_klib:LTC7106 U?
+U 1 1 5EC52C41
+P 4850 1700
+F 0 "U?" H 4500 2150 50  0000 C CNN
+F 1 "LTC7106" H 4850 1800 50  0000 C CNN
+F 2 "" H 4850 1700 50  0001 C CNN
+F 3 "" H 4850 1700 50  0001 C CNN
+	1    4850 1700
+	1    0    0    -1
+$EndComp
+Wire Wire Line
+	4750 900  4850 900
+Wire Wire Line
+	4850 1200 4850 900
+Connection ~ 4850 900
+Wire Wire Line
+	4850 900  5200 900
+$Comp
+L pps_klib:LTC7106 U?
+U 1 1 5EC55148
+P 4850 3850
+F 0 "U?" H 4500 4300 50  0000 C CNN
+F 1 "LTC7106" H 4850 3950 50  0000 C CNN
+F 2 "" H 4850 3850 50  0001 C CNN
+F 3 "" H 4850 3850 50  0001 C CNN
+	1    4850 3850
+	1    0    0    -1
+$EndComp
+$Comp
+L pps_klib:LTC7106 U?
+U 1 1 5EC55232
+P 4900 6000
+F 0 "U?" H 4550 6450 50  0000 C CNN
+F 1 "LTC7106" H 4900 6100 50  0000 C CNN
+F 2 "" H 4900 6000 50  0001 C CNN
+F 3 "" H 4900 6000 50  0001 C CNN
+	1    4900 6000
+	1    0    0    -1
+$EndComp

Commit message: lots of work
expanded README doc, specifications, added secondary regulator circuit + symbol, more component specs added
Parts:
- added TP?: GND, TestPoint:TestPoint_Keystone_5000-5004_Miniature, symbol Connector:TestPoint
- C?: footprint (none) -> Resistor_SMD:R_1210_3225Metric_Pad1.42x2.65mm_HandSolder
- R?: value 10 -> 0; Size (none) -> 0603
Connections:
- net GND: now also TP?.1
Other:
- note added: "REDO THIS CIRCUIT"
Changed lines of the file:
@@
 U 1 1 5E9697E8
 P 2000 3350
-F 0 "R?" V 1795 3350 50  0000 C CNN
-F 1 "10" V 1886 3350 50  0000 C CNN
+F 0 "R?" V 1700 3350 50  0000 C CNN
+F 1 "0" V 1800 3350 50  0000 C CNN
 F 2 "Resistor_SMD:R_0805_2012Metric" V 2040 3340 50  0001 C CNN
 F 3 "~" H 2000 3350 50  0001 C CNN
+F 4 "0603" V 1900 3350 50  0000 C CNN "Size"
 	1    2000 3350
 	0    1    1    0
@@
 F 0 "C?" H 2350 3700 50  0000 L CNN
 F 1 "22u" H 2350 3600 50  0000 L CNN
-F 2 "" H 2288 3500 50  0001 C CNN
+F 2 "Resistor_SMD:R_1210_3225Metric_Pad1.42x2.65mm_HandSolder" H 2288 3500 50  0001 C CNN
 F 3 "~" H 2250 3650 50  0001 C CNN
 F 4 "TDK_C3225X5R1C226K250AA" H 2250 3650 50  0001 C CNN "MfrNum"
@@
 	1    0    0    -1
 $EndComp
+Text Notes 8800 2200 0    100  ~ 0
+REDO THIS CIRCUIT
+$Comp
+L Connector:TestPoint TP?
+U 1 1 5ECDF7D7
+P 1750 1900
+AR Path="/5E80D1C0/5ECDF7D7" Ref="TP?"  Part="1"
+AR Path="/5E80D210/5ECDF7D7" Ref="TP?"  Part="1"
+AR Path="/5E84FADE/5ECDF7D7" Ref="TP?"  Part="1"
+AR Path="/5ECFB146/5ECDF7D7" Ref="TP?"  Part="1"
+AR Path="/5E918E7D/5ECDF7D7" Ref="TP?"  Part="1"
+F 0 "TP?" V 1750 2100 50  0000 L CNN
+F 1 "GND" V 1850 2100 50  0000 L CNN
+F 2 "TestPoint:TestPoint_Keystone_5000-5004_Miniature" H 1950 1900 50  0001 C CNN
+F 3 "~" H 1950 1900 50  0001 C CNN
+	1    1750 1900
+	0    1    1    0
+$EndComp
+Wire Wire Line
+	1750 1900 1650 1900
+Connection ~ 1650 1900
 $EndSCHEMATC

Commit message: more part numbers
Added manfacturer part numbers to ICs, added descriptions to symbols in library
Parts:
- removed U? (x2): LTC7106, symbol pps_klib:LTC7106
- added U? (x2): LTC7106, symbol pps_klib:LTC7106
- U?: MfrNum (none) -> ADI_LTC7106EDDB
Connections:
- net +5V: now also U?.3 (VDD), U?.3 (VDD), U?.9 (ASEL0)
- net EN_out: now also U?.7 (EN), U?.7 (EN)
- net GND: now also U?.10 (ASEL1), U?.10 (ASEL1), U?.11 (EP), U?.11 (EP), U?.5 (GND), U?.5 (GND)
- net Iout_adj: now also U?.6 (IDAC)
- net LDO_EN_A: now also U?.8 (GPO)
- net LDO_EN_B: now also U?.8 (GPO)
- net SCL: now also U?.2 (SCL), U?.2 (SCL)
- net SDA: now also U?.1 (SDA), U?.1 (SDA)
- net Vout_adj: now also U?.6 (IDAC)
- net ~ALT_2C: now also U?.4 (~ALERT)
- net ~ALT_2E: now also U?.4 (~ALERT)
Changed lines of the file:
@@
 F 2 "" H 4850 1700 50  0001 C CNN
 F 3 "" H 4850 1700 50  0001 C CNN
+F 4 "ADI_LTC7106EDDB" H 4850 1700 50  0001 C CNN "MfrNum"
 	1    4850 1700
 	1    0    0    -1
@@
 Wire Wire Line
 	4850 900  5200 900
-$Comp
-L pps_klib:LTC7106 U?
-U 1 1 5EC55148
-P 4850 3850
-F 0 "U?" H 4500 4300 50  0000 C CNN
-F 1 "LTC7106" H 4850 3950 50  0000 C CNN
-F 2 "" H 4850 3850 50  0001 C CNN
-F 3 "" H 4850 3850 50  0001 C CNN
-	1    4850 3850
-	1    0    0    -1
-$EndComp
-$Comp
-L pps_klib:LTC7106 U?
-U 1 1 5EC55232
-P 4900 6000
-F 0 "U?" H 4550 6450 50  0000 C CNN
-F 1 "LTC7106" H 4900 6100 50  0000 C CNN
-F 2 "" H 4900 6000 50  0001 C CNN
-F 3 "" H 4900 6000 50  0001 C CNN
-	1    4900 6000
-	1    0    0    -1
-$EndComp
 Text Notes 8800 2200 0    100  ~ 0
 REDO THIS CIRCUIT
@@
 	1750 1900 1650 1900
 Connection ~ 1650 1900
+$Comp
+L pps_klib:LTC7106 U?
+U 1 1 5ECC744C
+P 4850 3850
+F 0 "U?" H 4500 4300 50  0000 C CNN
+F 1 "LTC7106" H 4850 3950 50  0000 C CNN
+F 2 "" H 4850 3850 50  0001 C CNN
+F 3 "" H 4850 3850 50  0001 C CNN
+F 4 "ADI_LTC7106EDDB" H 4850 3850 50  0001 C CNN "MfrNum"
+	1    4850 3850
+	1    0    0    -1
+$EndComp
+$Comp
+L pps_klib:LTC7106 U?
+U 1 1 5ECC74B2
+P 4900 6000
+F 0 "U?" H 4550 6450 50  0000 C CNN
+F 1 "LTC7106" H 4900 6100 50  0000 C CNN
+F 2 "" H 4900 6000 50  0001 C CNN
+F 3 "" H 4900 6000 50  0001 C CNN
+F 4 "ADI_LTC7106EDDB" H 4900 6000 50  0001 C CNN "MfrNum"
+	1    4900 6000
+	1    0    0    -1
+$EndComp
 $EndSCHEMATC
