File: hw/design/SupplyAdj.sch (KiCad schematic (older format))
At the start: 17 parts

Commit message: reworked adjusters
new V/I adjustment scheme; modified LDO circuit to match
Parts:
- removed C? (x2): 1u, Resistor_SMD:R_0805_2012Metric_Pad1.15x1.40mm_HandSolder, symbol Device:C
- removed Q? (x2): DualPMOS, symbol Device:Q_DUAL_PMOS_G1S2G2D2S1D1
- removed R?: 0, Resistor_SMD:R_0805_2012Metric, symbol Device:R_US
- removed R? (x3): 100k, Resistor_SMD:R_0402_1005Metric, symbol Device:R_US
- removed U?: LTC7106, symbol pps_klib:LTC7106
- added C? (x5): 1u, Resistor_SMD:R_0805_2012Metric_Pad1.15x1.40mm_HandSolder, symbol Device:C
- added C?: 10n, Resistor_SMD:R_0603_1608Metric, symbol Device:C
- added R? (x8): 0, Resistor_SMD:R_0603_1608Metric, symbol Device:R_US
- added R?: 260k, Resistor_SMD:R_1206_3216Metric_Pad1.42x1.75mm_HandSolder, symbol Device:R_US
- added U? (x2): AD5272BRM, Package_SO:MSOP-10_3x3mm_P0.5mm, symbol Potentiometer_Digital:AD5272BRM
Connections:
- net EN_bus is gone; now on net +5V: U?.7 (EN)
- net +5V: now also C?.2, FB?.1, C?.2, C?.2, C?.2, R?.2, R?.2, R?.2, U?.1 (VDD), U?.1 (VDD); no longer U?.9 (ASEL0)
- net GND: now also C?.1, C?.1, C?.1, C?.1, C?.1, R?.2, R?.2, R?.2, R?.2, U?.3 (W), U?.4 (VSS), U?.4 (VSS), U?.6 (GND), U?.6 (GND); no longer U?.10 (ASEL1), U?.10 (ASEL1), U?.9 (ASEL0)
- net Iout_adj: now also U?.2 (A)
- net SCL: now also U?.9 (SCL), U?.9 (SCL)
- net SDA: now also U?.8 (SDA), U?.8 (SDA)
- net EN_out renamed DAC_en
- net LDO_EN_A renamed LDO_en
- net Vbus_adj renamed Vpre_adj
- net Vout_adj renamed LDO_adj
- net LDO_adj: now also C?.2, U?.2 (A)
- net ~ALT_2A: no longer names the net of U?.4 (~ALERT)
- new net: R?.1, U?.10 (ASEL1) (x2)
- new net: R?.1, U?.9 (ASEL0) (x2)
- new net: R?.1, U?.10 (ADDR) (x2)
- new net: R?.2, U?.3 (W)
- new net: C?.2, U?.5 (EXT_CAP) (x2)
- new net: R?.1, U?.7 (~RESET) (x2)
- new net LDO_out: C?.1, R?.1
- no-connect marks 1 -> 3
Other:
- note added: "ADDR = 0x2F"
- note added: "Address Table (7-bit)\n--------------------\n0x2A - Switcher DAC Vout Adjust\n0x2C - LDO DAC Vout Adjust\n0x2E - LDO Digipot Vout Adjust\n0x2F - LDO Current Limit Adjust\n0x57 - Global DAC Address\n0x58 - Global DAC Address"
- note added: "LDO Current\nLimit Adj."
- note added: "LDO Output\nVoltage Adj."
- note added: "Preregulator\nVoltage Adj"
- note added: "This resistor and digipot are\npart of the LDO feedback\ncircuit and should be laid\nout as such on the PCB"
- note removed: "Address Table (7-bit)\n--------------------\n0x2A - Switcher Vout Adjust\n0x2C - LDO Vout Adjust\n0x2E - LDO Iout Lim Adjust\n0x57 - Global Address\n0x58 - Global Address"
- note removed: "LDO Enable Circuitry"
- note removed: "LDO Output\nCurrent Limit\nAdjustment"
- note removed: "LDO Output\nVoltage Adjustment"
- note removed: "Preregulator Output\nVoltage Adjustment"
- note removed: "REDO THIS CIRCUIT"
- moved on the sheet: C?, U?
